Commit message: update files & upload

File: src/allegro_hand_controllers/urdf/allegro_hand_description_right.urdf (robot description, URDF)
Before this commit: robot allegro_hand_right, 35 links, 34 joints
Joints:
- joint joint_0_0: limit lower=-0.3 upper=0.3 effort=15 velocity=7 -> lower=-0.7 upper=0.262 effort=15 velocity=7
- joint joint_11_0: limit lower=-0.1 upper=2.01 effort=15 velocity=7 -> lower=-0.1 upper=1.86 effort=15 velocity=7
- joint joint_1_0: origin xyz=0 -0.000 0.03296 -> xyz=0 -0.000 0.03546
- joint joint_3_0: limit lower=-0.1 upper=2.01 effort=15 velocity=7 -> lower=-0.1 upper=1.86 effort=15 velocity=7
- joint joint_4_0: limit lower=-0.3 upper=0.3 effort=15 velocity=7 -> lower=-0.262 upper=0.262 effort=15 velocity=7
- joint joint_5_0: origin xyz=0 -0.000 0.03296 -> xyz=0 -0.000 0.03546
- joint joint_7_0: limit lower=-0.1 upper=2.01 effort=15 velocity=7 -> lower=-0.1 upper=1.86 effort=15 velocity=7
- joint joint_8_0: limit lower=-0.3 upper=0.3 effort=15 velocity=7 -> lower=-0.262 upper=0.7 effort=15 velocity=7
- joint joint_9_0: origin xyz=0 -0.000 0.03296 -> xyz=0 -0.000 0.03546
