Commit message: fix minor issues

File: src/allegro_hand_controllers/urdf/allegro_hand_description_left.urdf (robot description, URDF)
Before this commit: robot allegro_hand_left, 35 links, 34 joints
Joints:
- joint joint_1_0: origin xyz=0 -0.000 0.03296 -> xyz=0 -0.000 0.03546
- joint joint_5_0: origin xyz=0 -0.000 0.03296 -> xyz=0 -0.000 0.03546
- joint joint_9_0: origin xyz=0 -0.000 0.03296 -> xyz=0 -0.000 0.03546

Commit message: Update allegro_hand_description_left.urdf
Change left Hand thumb joint limit

File: src/allegro_hand_controllers/urdf/allegro_hand_description_left.urdf (robot description, URDF)
Before this commit: robot allegro_hand_left, 35 links, 34 joints
Joints:
- joint joint_12_0: limit lower=0.00 upper=1.78 effort=15 velocity=7 -> lower=-1.78 upper=0.00 effort=15 velocity=7
- joint joint_13_0: limit lower=-0.26 upper=1.78 effort=15 velocity=7 -> lower=1.78 upper=3.14 effort=15 velocity=7
- joint joint_14_0: limit lower=-0.05 upper=1.85 effort=15 velocity=7 -> lower=-1.78 upper=0.26 effort=15 velocity=7
- joint joint_15_0: limit lower=-0.09 upper=1.80 effort=15 velocity=7 -> lower=-1.80 upper=0.09 effort=15 velocity=7
